Commit message: modifed cmake of bringup pkg, changed hz from 1 to 100, found wheel seperation misconfiguration in controller.launch file, removed comments from cpp and py versions of simple_controller, updated the small_warehouse.world file to match antonio's, removed uart_test as it is not needed, added comments in bumperbot_ros2_control.xacro

File: src/bumperbot_description/urdf/bumperbot_ros2_control.xacro (robot description, xacro)
@@ -2,6 +2,6 @@
 <robot xmlns:xacro="http://www.ros.org/wiki/xacro" name="bumperbot">
     <ros2_control name="RobotSystem" type="system">
+        <!-- ros2_control Gazebo -->
         <xacro:if value="$(arg is_sim)">
-            <!-- ros2_control Gazebo -->
             <!-- ROS 2 Humble -->
             <xacro:if value="$(arg is_ignition)">
@@ -17,4 +17,5 @@
             </xacro:unless>
         </xacro:if>
+        <!-- ros2_control Real Robot -->
         <xacro:unless value="$(arg is_sim)">
             <hardware>
@@ -24,5 +25,5 @@
         </xacro:unless>
         <!-- ros2_control Common Interfaces -->
-        <joint name="wheel_right_joint">
+        <joint name="wheel_left_joint">
             <command_interface name="velocity">
               <param name="min">-1</param>
@@ -32,5 +33,5 @@
             <state_interface name="velocity" />
         </joint>
-        <joint name="wheel_left_joint">
+        <joint name="wheel_right_joint">
             <command_interface name="velocity">
               <param name="min">-1</param>
