Commit message: made small changes

File: src/bumperbot_description/urdf/bumperbot.urdf.xacro (robot description, xacro)
@@ -159,5 +159,5 @@
           <mesh filename="package://bumperbot_description/meshes/new_laser_link.stl"/>
         </geometry>
-        <origin xyz="0 0 0" rpy="0 0 0"/>
+        <origin xyz="0 0 0" rpy="0 0 3.14"/>
         <material name="dark_grey"/>
       </visual>
@@ -170,5 +170,5 @@
     </link>
   <joint name="laser_joint" type="fixed">
-        <origin xyz="0 0 0.131" rpy="0 0 3.14" /> <!-- z= 0.042(from physical unit) + 0.088(from fusion final assembly without wheels) + 0.001(accounting for plate thickness)-->
+        <origin xyz="0 0 0.131" rpy="0 0 0" /> <!-- z= 0.042(from physical unit) + 0.088(from fusion final assembly without wheels) + 0.001(accounting for plate thickness)-->
         <parent link="base_link" />
         <child link="laser_link" />

Commit message: tested code in rviz, working

File: src/bumperbot_description/urdf/bumperbot.urdf.xacro (robot description, xacro)
@@ -11,9 +11,9 @@
   <link name="base_link">
     <inertial>
-      <origin xyz="0.000392694 0.003603923 0.028354103" rpy="0 0 0"/>
-      <mass value="1.1796479"/>
-      <inertia ixx="0.010666756"    ixy="0.000115581"  ixz="0.001086391"
-               iyy="0.011710101"    iyz="-0.000017452"
-               izz="0.00663569" />
+      <origin xyz="-0.008675826 0.003144972 0.032628778" rpy="0 0 0"/>
+      <mass value="2.210665107"/>
+      <inertia ixx="0.011527704"    ixy="-5.335634932e-7"  ixz="-0.000228605"
+               iyy="0.005806872"    iyz="-0.000372021"
+               izz="0.014234404" />
     </inertial>
     <visual>
@@ -159,5 +159,5 @@
           <mesh filename="package://bumperbot_description/meshes/new_laser_link.stl"/>
         </geometry>
-        <origin xyz="0 0 0" rpy="0 0 3.14"/>
+        <origin xyz="0 0 0" rpy="0 0 0"/>
         <material name="dark_grey"/>
       </visual>
@@ -170,5 +170,5 @@
     </link>
   <joint name="laser_joint" type="fixed">
-        <origin xyz="0 0 0.131" rpy="0 0 0" /> <!-- z= 0.042(from physical unit) + 0.088(from fusion final assembly without wheels) + 0.001(accounting for plate thickness)-->
+        <origin xyz="0 0 0.131" rpy="0 0 3.14" /> <!-- z= 0.042(from physical unit) + 0.088(from fusion final assembly without wheels) + 0.001(accounting for plate thickness)-->
         <parent link="base_link" />
         <child link="laser_link" />

Commit message: modifed urdf, made final changes, assembly of robot in real life is done

File: src/bumperbot_description/urdf/bumperbot.urdf.xacro (robot description, xacro)
@@ -21,5 +21,5 @@
       <!-- <material name="black"/> -->
       <geometry>
-        <mesh filename="package://bumperbot_description/meshes/base_link.stl" scale="0.001 0.001 0.001"/>
+        <mesh filename="package://bumperbot_description/meshes/base_link.stl"/>
       </geometry>
     </visual>
@@ -27,5 +27,5 @@
       <origin xyz="0 0 0.0015" rpy="0 0 0" />
       <geometry>
-        <mesh filename="package://bumperbot_description/meshes/base_link.stl" scale="0.001 0.001 0.001"/>
+        <mesh filename="package://bumperbot_description/meshes/base_link.stl"/>
       </geometry>
     </collision>
@@ -34,5 +34,5 @@
     <parent link="base_footprint"/>
     <child link="base_link" />
-    <origin xyz="0 0 0.038" rpy="0 0 0"/>
+    <origin xyz="0 0 0.02434923" rpy="0 0 0"/>
   </joint>
   <link name="wheel_right_link">
@@ -45,5 +45,5 @@
     </inertial>
     <visual>
-      <origin xyz="0 0 0" rpy="1.57 0 0" />
+      <origin xyz="0 0 0" rpy="-1.57 0 0" />
       <material name="blue" />
       <geometry>
@@ -58,13 +58,12 @@
     </collision>
   </link>
-  <joint name="wheel_right_joint" type="continuous">
-    <origin xyz="0 -0.11455 0.015" rpy="0 0 0" />
+   <joint name="wheel_right_joint" type="continuous">
+    <origin xyz="0 0.14513032 0.03" rpy="0 0 0" />
     <parent link="base_link" />
     <child link="wheel_right_link" />
     <axis xyz="0 1 0" />
   </joint>
-  <link
-    name="wheel_left_link">
-    <inertial>
+  <link name="wheel_left_link">
+   <inertial>
       <origin xyz="0 9.713661142e-10 0.016398450" rpy="0 0 0" />
       <mass value="0.092049771" />
@@ -74,12 +73,12 @@
     </inertial>
     <visual>
-      <origin xyz="0 0 0" rpy="-1.57 0 0" />
+      <origin xyz="0 0 0" rpy="1.57 0 0" />
       <material name="blue" />
       <geometry>
-        <mesh filename="package://bumperbot_description/meshes/wheel_left_link.stl"/>
-      </geometry>
-    </visual>
-    <collision>
-      <origin xyz="0 0.017 0" rpy="-1.57 0 0" />
+        <mesh filename="package://bumperbot_description/meshes/wheel_right_link.stl"/>
+      </geometry>
+    </visual>
+    <collision>
+      <origin xyz="0 -0.017 0" rpy="1.57 0 0" />
       <geometry>
         <cylinder radius="0.0534" length="0.0285"/>
@@ -87,6 +86,6 @@
     </collision>
   </link>
-  <joint name="wheel_left_joint" type="continuous">
-    <origin xyz="0 0.11455 0.015" rpy="0 0 0" />
+   <joint name="wheel_left_joint" type="continuous">
+    <origin xyz="0 -0.14513032 0.03" rpy="0 0 0" />
     <parent link="base_link" />
     <child link="wheel_left_link" />
@@ -95,12 +94,12 @@
   <link name="caster_front_link">
     <inertial>
-      <origin xyz="-0.055462489 0.004963490 0.019704843" rpy="0 0 0" />
-      <mass value="0.034768653" />
-      <inertia ixx="0.000006952"  ixy="-8.168396889e-10"    ixz="4.36638148e-10"
-               iyy="0.00000631"  iyz="-8.101927285e-10"
-               izz="0.000006556" />
-    </inertial>
-    <visual>
-      <origin xyz="0 0 0" rpy="0 0 1.57" />
+      <origin xyz="5.375138993e-07 -9.84538264e-07 0.012447006" rpy="0 0 0" />
+      <mass value="0.006654822" />
+      <inertia ixx="5.314741443e-07"  ixy="0.00"    ixz="0.00"
+               iyy="4.867361117e-07"  iyz="0.00"
+               izz="4.568100217e-07" />
+    </inertial>
+    <visual>
+      <origin xyz="0 0 0" rpy="0 0 0" />
       <material name="silver"/>
       <geometry>
@@ -109,5 +108,5 @@
     </visual>
     <collision>
-      <origin xyz="0 0 0.0211305" rpy="0 0 1.57" />
+      <origin xyz="0 0 0.0211305" rpy="0 0 0" />
       <geometry>
         <sphere radius="0.0211305"/>
@@ -116,5 +115,5 @@
   </link>
   <joint name="caster_front_joint" type="fixed">
-    <origin xyz="0.0762 0 -0.0380011" rpy="0 0 0" />
+    <origin xyz="0.1101000 0.00074129 -0.02400923" rpy="0 0 0" />
     <parent link="base_link" />
     <child link="caster_front_link" />
@@ -122,12 +121,12 @@
   <link name="caster_rear_link">
     <inertial>
-      <origin xyz="-0.055462489 0.004963490 0.019704843" rpy="0 0 0" />
-      <mass value="0.034768653" />
-      <inertia ixx="0.000006952"  ixy="-8.168396889e-10"    ixz="4.36638148e-10"
-               iyy="0.00000631"  iyz="-8.101927285e-10"
-               izz="0.000006556" />
-    </inertial>
-    <visual>
-      <origin xyz="0 0 0" rpy="0 0 1.57" />
+      <origin xyz="5.375138993e-07 -9.84538264e-07 0.012447006" rpy="0 0 0" />
+      <mass value="0.006654822" />
+      <inertia ixx="5.314741443e-07"  ixy="0.00"    ixz="0.00"
+               iyy="4.867361117e-07"  iyz="0.00"
+               izz="4.568100217e-07" />
+    </inertial>
+    <visual>
+      <origin xyz="0 0 0" rpy="0 0 0" />
       <material name="silver"/>
       <geometry>
@@ -136,5 +135,5 @@
     </visual>
     <collision>
-      <origin xyz="0 0 0.0211305" rpy="0 0 1.57" />
+      <origin xyz="0 0 0.0211305" rpy="0 0 0" />
       <geometry>
         <sphere radius="0.0211305"/>
@@ -143,5 +142,5 @@
   </link>
   <joint name="caster_rear_joint" type="fixed">
-    <origin xyz="-0.0762 0 -0.0380011" rpy="0 0 0" />
+    <origin xyz="-0.1101000 0.00074129 -0.02400923" rpy="0 0 0" />
     <parent link="base_link" />
     <child link="caster_rear_link" />
@@ -152,10 +151,10 @@
         <mass value="0.1700"/>
         <inertia ixx="7.403494e-05"  ixy="5.337393e-06"  ixz="1.511932e-05"
-                                        iyy="1.426408e-04"  iyz="1.752534e-06"
+                                     iyy="1.426408e-04"  iyz="1.752534e-06"
                                                             izz="1.672852e-04"/>
       </inertial>
       <visual>
         <geometry>
-          <mesh filename="package://bumperbot_description/meshes/new_laser_link.stl"/>
+          <mesh filename="package://bumperbot_description/meshes/laser_link.stl"/>
         </geometry>
         <origin xyz="0 0 0" rpy="0 0 0"/>
@@ -166,9 +165,9 @@
           <box size="0.071689 0.097337 0.05350"/>
         </geometry>
-        <origin xyz="0 0 -0.015" rpy="0 0 0"/>
+        <origin xyz="0 0 0" rpy="0 0 0"/>
       </collision>
     </link>
   <joint name="laser_joint" type="fixed">
-        <origin xyz="0 0 0.131" rpy="0 0 3.14" /> <!-- z= 0.042(from physical unit) + 0.088(from fusion final assembly without wheels) + 0.001(accounting for plate thickness)-->
+       <origin xyz="0 0 0.109" rpy="0 0 0" /> <!--z= 0.042(from physical unit) + 0.088(from fusion final assembly without wheels) + 0.001(accounting for plate thickness)-->
         <parent link="base_link" />
         <child link="laser_link" />
@@ -184,5 +183,5 @@
       <material name="amber_gold"/>
       <geometry>
-        <mesh filename="package://bumperbot_description/meshes/imu_link.STL"/>
+        <mesh filename="package://bumperbot_description/meshes/imu_link_new.stl"/>
       </geometry>
     </visual>
@@ -197,5 +196,5 @@
     <parent link="base_link"/>
     <child link="imu_link"/>
-    <origin xyz="-0.020000 -0.08000 0.04780000" rpy="0.0 0.0 0.0"/> <!-- x and y values from fusion and z value is from fusion but also adjusted-->
+  <origin xyz="0.0 0.008 0.07" rpy="0.0 0.0 0.0"/> <!--x and y values from fusion and z value is from fusion but also adjusted -->
   </joint>
   <material name="blue">

Commit message: modified urdf, tuned collision data, robot not running in gazebo, fixing

File: src/bumperbot_description/urdf/bumperbot.urdf.xacro (robot description, xacro)
@@ -52,5 +52,5 @@
     </visual>
     <collision>
-      <origin xyz="0 -0.017 0" rpy="1.57 0 0" />
+      <origin xyz="0 0.0174 0" rpy="1.57 0 0" />
       <geometry>
         <cylinder radius="0.0534" length="0.0285"/>
@@ -64,6 +64,7 @@
     <axis xyz="0 1 0" />
   </joint>
-  <link name="wheel_left_link">
-   <inertial>
+  <link
+    name="wheel_left_link">
+    <inertial>
       <origin xyz="0 9.713661142e-10 0.016398450" rpy="0 0 0" />
       <mass value="0.092049771" />
@@ -76,9 +77,9 @@
       <material name="blue" />
       <geometry>
-        <mesh filename="package://bumperbot_description/meshes/wheel_right_link.stl"/>
-      </geometry>
-    </visual>
-    <collision>
-      <origin xyz="0 -0.017 0" rpy="1.57 0 0" />
+        <mesh filename="package://bumperbot_description/meshes/wheel_left_link.stl"/>
+      </geometry>
+    </visual>
+    <collision>
+      <origin xyz="0 -0.0174 0" rpy="1.57 0 0" />
       <geometry>
         <cylinder radius="0.0534" length="0.0285"/>
@@ -108,12 +109,12 @@
     </visual>
     <collision>
-      <origin xyz="0 0 0.0211305" rpy="0 0 0" />
-      <geometry>
-        <sphere radius="0.0211305"/>
+      <origin xyz="0 0 0.01240923" rpy="0 0 0" />
+      <geometry>
+        <sphere radius="0.013004615"/>
       </geometry>
     </collision>
   </link>
   <joint name="caster_front_joint" type="fixed">
-    <origin xyz="0.1101000 0.00074129 -0.02400923" rpy="0 0 0" />
+    <origin xyz="0.1101000 0.00074129 -0.02450923" rpy="0 0 0" />
     <parent link="base_link" />
     <child link="caster_front_link" />
@@ -135,12 +136,12 @@
     </visual>
     <collision>
-      <origin xyz="0 0 0.0211305" rpy="0 0 0" />
-      <geometry>
-        <sphere radius="0.0211305"/>
+      <origin xyz="0 0 0.01240923" rpy="0 0 0" />
+      <geometry>
+        <sphere radius="0.013004615"/>
       </geometry>
     </collision>
   </link>
   <joint name="caster_rear_joint" type="fixed">
-    <origin xyz="-0.1101000 0.00074129 -0.02400923" rpy="0 0 0" />
+    <origin xyz="-0.1101000 0.00074129 -0.02450923" rpy="0 0 0" />
     <parent link="base_link" />
     <child link="caster_rear_link" />
@@ -158,14 +159,14 @@
           <mesh filename="package://bumperbot_description/meshes/laser_link.stl"/>
         </geometry>
-        <origin xyz="0 0 0" rpy="0 0 0"/>
+        <origin xyz="0 0 0" rpy="0 0 3.14"/>
         <material name="dark_grey"/>
       </visual>
       <collision>
+        <origin xyz="0 0 0.03150" rpy="0 0 3.14"/>
         <geometry>
           <box size="0.071689 0.097337 0.05350"/>
         </geometry>
-        <origin xyz="0 0 0" rpy="0 0 0"/>
       </collision>
-    </link>
+  </link>
   <joint name="laser_joint" type="fixed">
        <origin xyz="0 0 0.109" rpy="0 0 0" /> <!--z= 0.042(from physical unit) + 0.088(from fusion final assembly without wheels) + 0.001(accounting for plate thickness)-->

Commit message: found error, wheel not touching

File: src/bumperbot_description/urdf/bumperbot.urdf.xacro (robot description, xacro)
@@ -45,5 +45,5 @@
     </inertial>
     <visual>
-      <origin xyz="0 0 0" rpy="-1.57 0 0" />
+      <origin xyz="0 0 0" rpy="1.57 0 0" />
       <material name="blue" />
       <geometry>
@@ -52,5 +52,5 @@
     </visual>
     <collision>
-      <origin xyz="0 0.0174 0" rpy="1.57 0 0" />
+      <origin xyz="0 -0.0146 0" rpy="1.57 0 0" />
       <geometry>
         <cylinder radius="0.0534" length="0.0285"/>
@@ -59,5 +59,5 @@
   </link>
    <joint name="wheel_right_joint" type="continuous">
-    <origin xyz="0 0.14513032 0.03" rpy="0 0 0" />
+    <origin xyz="0 0.16513032 0.035" rpy="0 0 0" />
     <parent link="base_link" />
     <child link="wheel_right_link" />
@@ -74,5 +74,5 @@
     </inertial>
     <visual>
-      <origin xyz="0 0 0" rpy="1.57 0 0" />
+      <origin xyz="0 0 0" rpy="-1.57 0 0" />
       <material name="blue" />
       <geometry>
@@ -81,5 +81,5 @@
     </visual>
     <collision>
-      <origin xyz="0 -0.0174 0" rpy="1.57 0 0" />
+      <origin xyz="0 0.0146 0" rpy="-1.57 0 0" />
       <geometry>
         <cylinder radius="0.0534" length="0.0285"/>
@@ -88,5 +88,5 @@
   </link>
    <joint name="wheel_left_joint" type="continuous">
-    <origin xyz="0 -0.14513032 0.03" rpy="0 0 0" />
+    <origin xyz="0 -0.16513032 0.035" rpy="0 0 0" />
     <parent link="base_link" />
     <child link="wheel_left_link" />
@@ -102,5 +102,5 @@
     </inertial>
     <visual>
-      <origin xyz="0 0 0" rpy="0 0 0" />
+      <origin xyz="0 0 0" rpy="0 0 1.57" />
       <material name="silver"/>
       <geometry>
@@ -109,5 +109,5 @@
     </visual>
     <collision>
-      <origin xyz="0 0 0.01240923" rpy="0 0 0" />
+      <origin xyz="0 0 0.01240923" rpy="0 0 1.57" />
       <geometry>
         <sphere radius="0.013004615"/>
@@ -129,5 +129,5 @@
     </inertial>
     <visual>
-      <origin xyz="0 0 0" rpy="0 0 0" />
+      <origin xyz="0 0 0" rpy="0 0 1.57" />
       <material name="silver"/>
       <geometry>
@@ -136,5 +136,5 @@
     </visual>
     <collision>
-      <origin xyz="0 0 0.01240923" rpy="0 0 0" />
+      <origin xyz="0 0 0.01240923" rpy="0 0 1.57" />
       <geometry>
         <sphere radius="0.013004615"/>
